Commit message: change in URDF

File: omni_description/urdf/omni_table.urdf (robot description, URDF)
Before this commit: robot phantom_omni, 2 links, 2 joints
Links:
- removed link box
- added link base; visual mesh filename=package://omni_description/meshes/base.stl
- added link box2, mass 2.0; collision box size=1.0 1.0 1.0; visual box size=1.0 1.0 1.0
- added link end_effector
- added link lower_arm; visual mesh filename=package://omni_description/meshes/lower_arm.stl
- added link stylus; visual mesh filename=package://omni_description/meshes/pen.stl
- added link tip; visual mesh filename=package://omni_description/meshes/tip.stl
- added link torso; visual mesh filename=package://omni_description/meshes/torso.stl
- added link upper_arm; visual mesh filename=package://omni_description/meshes/upper_arm.stl
- added link wrist; visual mesh filename=package://omni_description/meshes/wrist.stl
Joints:
- removed joint box_to_base
- removed joint world_to_box
- added joint box2_to_base: type fixed, parent box2, child base, origin xyz=0 0 1 rpy=0 0 0
- added joint effector_transform: type fixed, parent tip, child end_effector, origin xyz=0 0.031 0 rpy=0 0 0
- added joint elbow: type revolute, parent upper_arm, child lower_arm, origin xyz=0.0075 .134 0 rpy=-2.15 0 0, axis 1 0 0, limit lower=-0.2 upper=1.95 effort=5 velocity=100
- added joint shoulder: type revolute, parent torso, child upper_arm, origin xyz=-0.0075 0 0.035 rpy=0.23 0 0, axis 1 0 0, limit lower=-0.24 upper=1.57 effort=5 velocity=100
- added joint waist: type revolute, parent base, child torso, origin xyz=0 0 0.09 rpy=0 0 0, axis 0 0 1, limit lower=-0.98 upper=0.98 effort=5 velocity=100
- added joint world_to_box2: type fixed, parent world, child box2
- added joint wrist1: type revolute, parent lower_arm, child wrist, origin xyz=0 0.08 0 rpy=0 0 0, axis 0 1 0, limit lower=-2.54 upper=2.60 effort=5 velocity=100
- added joint wrist2: type revolute, parent wrist, child tip, origin xyz=0 0.0525 0 rpy=-0.85 0 0, axis 1 0 0, limit lower=-2.07 upper=0.23 effort=5 velocity=100
- added joint wrist3: type revolute, parent tip, child stylus, origin xyz=0 -0.023 0 rpy=0 0 0, axis 0 1 0, limit lower=-2.34 upper=2.34 effort=5 velocity=100
