Commit message: changing the moveit setup for the omni_phantom

File: omni_description/urdf/omni.urdf (robot description, URDF)
Before this commit: robot phantom_omni, 8 links, 7 joints
Links:
- link base: mass None -> 0.3; geometry collision mesh filename=package://omni_description/meshes/base.stl; visual mesh filename=package://omni_description/meshes/base.stl
- link lower_arm: mass None -> 0.1; geometry collision mesh filename=package://omni_description/meshes/lower_arm.stl; visual mesh filename=package://omni_description/meshes/lower_arm.stl
- link stylus: mass None -> 0.1; geometry collision mesh filename=package://omni_description/meshes/pen.stl; visual mesh filename=package://omni_description/meshes/pen.stl
- link tip: mass None -> 0.1; geometry collision mesh filename=package://omni_description/meshes/tip.stl; visual mesh filename=package://omni_description/meshes/tip.stl
- link torso: mass None -> 0.2; geometry collision mesh filename=package://omni_description/meshes/torso.stl; visual mesh filename=package://omni_description/meshes/torso.stl
- link upper_arm: mass None -> 0.1; geometry collision mesh filename=package://omni_description/meshes/upper_arm.stl; visual mesh filename=package://omni_description/meshes/upper_arm.stl
- link wrist: mass None -> 0.2; geometry collision mesh filename=package://omni_description/meshes/wrist.stl; visual mesh filename=package://omni_description/meshes/wrist.stl

File: omni_description/urdf/omni_table.urdf (robot description, URDF)
Before this commit: robot phantom, 10 links, 9 joints
Links:
- link base: mass None -> 0.3; geometry collision mesh filename=package://omni_description/meshes/base.stl; visual mesh filename=package://omni_description/meshes/base.stl
- link lower_arm: mass None -> 0.1; geometry collision mesh filename=package://omni_description/meshes/lower_arm.stl; visual mesh filename=package://omni_description/meshes/lower_arm.stl
- link stylus: mass None -> 0.1; geometry collision mesh filename=package://omni_description/meshes/pen.stl; visual mesh filename=package://omni_description/meshes/pen.stl
- link tip: mass None -> 0.1; geometry collision mesh filename=package://omni_description/meshes/tip.stl; visual mesh filename=package://omni_description/meshes/tip.stl
- link torso: mass None -> 0.2; geometry collision mesh filename=package://omni_description/meshes/torso.stl; visual mesh filename=package://omni_description/meshes/torso.stl
- link upper_arm: mass None -> 0.1; geometry collision mesh filename=package://omni_description/meshes/upper_arm.stl; visual mesh filename=package://omni_description/meshes/upper_arm.stl
- link wrist: mass None -> 0.2; geometry collision mesh filename=package://omni_description/meshes/wrist.stl; visual mesh filename=package://omni_description/meshes/wrist.stl
Joints:
- joint world_to_box2: origin (none) -> xyz=0 2 0 rpy=0 0 0
